Commit message: final

File: temp_mountain_0.urdf (robot description, URDF)
Before this commit: robot pepe, 1 links, 0 joints
Links:
- added link 11, mass 0.32542964784039335; collision cylinder length=1.7939906307955067 radius=0.24029433729724395; visual cylinder length=1.7939906307955067 radius=0.24029433729724395
- added link 22, mass 0.3456387518987746; collision cylinder length=1.7402814386779732 radius=0.2514354642671235; visual cylinder length=1.7402814386779732 radius=0.2514354642671235
- added link 23, mass 0.3456387518987746; collision cylinder length=1.7402814386779732 radius=0.2514354642671235; visual cylinder length=1.7402814386779732 radius=0.2514354642671235
- added link 24, mass 0.3456387518987746; collision cylinder length=1.7402814386779732 radius=0.2514354642671235; visual cylinder length=1.7402814386779732 radius=0.2514354642671235
- added link 35, mass 0.0026818171007753355; collision cylinder length=1.337972422484723 radius=0.025258994624506426; visual cylinder length=1.337972422484723 radius=0.025258994624506426
- added link 36, mass 0.0026818171007753355; collision cylinder length=1.337972422484723 radius=0.025258994624506426; visual cylinder length=1.337972422484723 radius=0.025258994624506426
- added link 37, mass 0.0026818171007753355; collision cylinder length=1.337972422484723 radius=0.025258994624506426; visual cylinder length=1.337972422484723 radius=0.025258994624506426
- link 0: mass 5.672400887905702 -> 0.07870743487701207; geometry collision cylinder length=0.41703708533247724 radius=0.24510129433127736; visual cylinder length=0.41703708533247724 radius=0.24510129433127736
Joints:
- added joint 11_to_0: type revolute, parent 0, child 11, origin xyz=0.3684942285678249 0.47884957059801336 0.8017108469487813 rpy=6.897320077721064 2.2458082970001523 3.4178430874805397, axis 0 1 0, limit lower=3.1415 upper=-3.1415 effort=1 velocity=1
- added joint 22_to_11: type revolute, parent 11, child 22, origin xyz=0.7520576552854916 0.787909909003156 0.9858630834839593 rpy=3.5307818349792965 2.5065007603570355 4.342087598570308, axis 1 0 0, limit lower=3.1415 upper=-3.1415 effort=1 velocity=1
- added joint 23_to_11: type revolute, parent 11, child 23, origin xyz=0.7520576552854916 0.787909909003156 0.9858630834839593 rpy=5.296172752468944 2.5065007603570355 4.342087598570308, axis 1 0 0, limit lower=3.1415 upper=-3.1415 effort=1 velocity=1
- added joint 24_to_11: type revolute, parent 11, child 24, origin xyz=0.7520576552854916 0.787909909003156 0.9858630834839593 rpy=7.061563669958593 2.5065007603570355 4.342087598570308, axis 1 0 0, limit lower=3.1415 upper=-3.1415 effort=1 velocity=1
- added joint 35_to_0: type revolute, parent 0, child 35, origin xyz=0.6345604679540542 0.1174361008392818 0.7225051083317479 rpy=5.866666503067048 1.7977758134575648 5.593589069951501, axis 0 0 1, limit lower=3.1415 upper=-3.1415 effort=1 velocity=1
- added joint 36_to_0: type revolute, parent 0, child 36, origin xyz=0.6345604679540542 0.1174361008392818 0.7225051083317479 rpy=7.822222004089397 1.7977758134575648 5.593589069951501, axis 0 0 1, limit lower=3.1415 upper=-3.1415 effort=1 velocity=1
- added joint 37_to_0: type revolute, parent 0, child 37, origin xyz=0.6345604679540542 0.1174361008392818 0.7225051083317479 rpy=9.777777505111747 1.7977758134575648 5.593589069951501, axis 0 0 1, limit lower=3.1415 upper=-3.1415 effort=1 velocity=1
