Commit message: first

File: temp_mountain_1.urdf (robot description, URDF)
Before this commit: robot pepe, 1 links, 0 joints
Links:
- link 0: mass 1.2015885542306328 -> 5.325411038520067; geometry collision cylinder length=1.9998 radius=0.920679236108968; visual cylinder length=1.9998 radius=0.920679236108968

File: temp_mountain_2.urdf (robot description, URDF)
Before this commit: robot pepe, 16 links, 15 joints
Links:
- removed link 11
- removed link 15
- removed link 19
- removed link 213
- removed link 214
- removed link 215
- removed link 310
- removed link 311
- removed link 312
- removed link 32
- removed link 33
- removed link 34
- removed link 36
- removed link 37
- removed link 38
- link 0: mass 0.32542964784039335 -> 6.281300540076709; geometry collision cylinder length=1.9998 radius=0.9999; visual cylinder length=1.9998 radius=0.9999
Joints:
- removed joint 11_to_0
- removed joint 15_to_0
- removed joint 19_to_0
- removed joint 213_to_0
- removed joint 214_to_0
- removed joint 215_to_0
- removed joint 310_to_19
- removed joint 311_to_19
- removed joint 312_to_19
- removed joint 32_to_11
- removed joint 33_to_11
- removed joint 34_to_11
- removed joint 36_to_15
- removed joint 37_to_15
- removed joint 38_to_15

File: temp_mountain_3.urdf (robot description, URDF)
Before this commit: robot pepe, 5 links, 4 joints
Links:
- removed link 22
- removed link 23
- removed link 24
- link 0: mass 0.3456387518987746 -> 5.325411038520067; geometry collision cylinder length=1.9998 radius=0.920679236108968; visual cylinder length=1.9998 radius=0.920679236108968
- link 11: mass 1.8835928743458918 -> 3.063990248021326; geometry collision cylinder length=1.3897543118212539 radius=0.8377216470649189; visual cylinder length=1.3897543118212539 radius=0.8377216470649189
Joints:
- removed joint 22_to_0
- removed joint 23_to_0
- removed joint 24_to_0
- joint 11_to_0: axis 0 0 1 -> 0 1 0; origin xyz=0.875913495298717 0.9648455558761536 0.3898030649287467 rpy=7.990417573566668 3.383946299899582 1.553446088233857 -> xyz=0.9802248488304317 0.576453298275668 0.714552166094369 rpy=8.963030129196884 4.258849670329692 0.6333811768262183

File: temp_viz.urdf (robot description, URDF)
Before this commit: robot pepe, 7 links, 6 joints
Links:
- removed link 24
- removed link 35
- removed link 36
- added link 14, mass 6.281300540076709; collision cylinder length=1.9998 radius=0.9999; visual cylinder length=1.9998 radius=0.9999
- added link 25, mass 1.8825643566191614; collision cylinder length=1.0088065689502967 radius=0.7707189348450902; visual cylinder length=1.0088065689502967 radius=0.7707189348450902
- added link 26, mass 1.8825643566191614; collision cylinder length=1.0088065689502967 radius=0.7707189348450902; visual cylinder length=1.0088065689502967 radius=0.7707189348450902
- link 0: mass 0.5172958498018503 -> 3.009762110778277; geometry collision cylinder length=1.9998 radius=0.6921462447369557; visual cylinder length=1.9998 radius=0.6921462447369557
- link 11: mass 1.015587507572395 -> 6.281300540076709; geometry collision cylinder length=1.9998 radius=0.9999; visual cylinder length=1.9998 radius=0.9999
- link 22: mass 0.009558088479673975 -> 1.8825643566191614; geometry collision cylinder length=1.0088065689502967 radius=0.7707189348450902; visual cylinder length=1.0088065689502967 radius=0.7707189348450902
- link 23: mass 0.009558088479673975 -> 1.8825643566191614; geometry collision cylinder length=1.0088065689502967 radius=0.7707189348450902; visual cylinder length=1.0088065689502967 radius=0.7707189348450902
Joints:
- removed joint 24_to_11
- removed joint 35_to_0
- removed joint 36_to_0
- added joint 14_to_0: type revolute, parent 0, child 14, origin xyz=0.38510891560579563 0.34321537469017627 0.08051966649087028 rpy=4.5166183713337675 6.282556988648868 0.23221567026121676, axis 1 0 0, limit lower=3.1415 upper=-3.1415 effort=1 velocity=1
- added joint 25_to_14: type revolute, parent 14, child 25, origin xyz=0.6465744440019845 0.3185629063362395 0.9856707806421344 rpy=12.565113977297736 4.130193121910501 4.541234158045601, axis 0 1 0, limit lower=3.1415 upper=-3.1415 effort=1 velocity=1
- added joint 26_to_14: type revolute, parent 14, child 26, origin xyz=0.6465744440019845 0.3185629063362395 0.9856707806421344 rpy=18.847670965946605 4.130193121910501 4.541234158045601, axis 0 1 0, limit lower=3.1415 upper=-3.1415 effort=1 velocity=1
- joint 11_to_0: axis 0 0 1 -> 1 0 0; origin xyz=0.36813298449497434 0.8011075333734261 0.1889147050062893 rpy=7.517099752517243 1.9967120255464816 5.1403467964114 -> xyz=0.38510891560579563 0.34321537469017627 0.08051966649087028 rpy=3.011078914222512 6.282556988648868 0.23221567026121676
- joint 22_to_11: axis 0 0 1 -> 0 1 0; origin xyz=0.6347812771404477 0.6119682614187647 0.3344417075701225 rpy=3.9995369568553443 1.743286167099876 1.4519012211936142 -> xyz=0.6465744440019845 0.3185629063362395 0.9856707806421344 rpy=12.565113977297736 4.130193121910501 4.541234158045601
- joint 23_to_11: axis 0 0 1 -> 0 1 0; origin xyz=0.6347812771404477 0.6119682614187647 0.3344417075701225 rpy=5.999305435283016 1.743286167099876 1.4519012211936142 -> xyz=0.6465744440019845 0.3185629063362395 0.9856707806421344 rpy=18.847670965946605 4.130193121910501 4.541234158045601
